Commit message: Updated mobile robot xacro

File: urdf/7_dof_arm.xacro (robot description, xacro)
@@ -56,9 +56,10 @@
   </joint>
   <link name="bottom_link">
-    <inertial>
+<!--    <inertial>
       <origin xyz=" 0 0 -0.017"/>
       <mass value="100.0" />
       <inertia  ixx="1.0" ixy="0.0"  ixz="0.0"  iyy="100.0"  iyz="0.0"  izz="1.0" />
     </inertial>
+-->
     <visual>
       <origin xyz=" 0 0 -0.04"  rpy="0 0 0"/>
@@ -69,5 +70,5 @@
     </visual>
     <collision>
-      <origin xyz=" 0 0 -0.017"  rpy="${.5*M_PI} 0 ${.5*M_PI}"/>
+      <origin xyz=" 0 0 -0.04"  rpy="0 0 0"/>
       <geometry>
 	       <box size="1 1 0.02" />
@@ -81,4 +82,5 @@
   <!-- BASE LINK -->
   <link name="base_link">
+<!--
     <inertial>
         <origin xyz="0 0 0" />
@@ -86,4 +88,5 @@
         <inertia  ixx="1.0" ixy="0.0"  ixz="0.0"  iyy="100.0"  iyz="0.0"  izz="1.0" />
         </inertial>
+-->
     <visual>
       <origin xyz="0 0 0" rpy="${M_PI/2} 0 0" /> <!-- rotate PI/2 -->
@@ -127,5 +130,5 @@
     </visual>
     <collision>
-      <origin xyz="0 0 0" rpy="0 0 ${M_PI/2}" />
+      <origin xyz="0 0 0" rpy="0 ${M_PI/2} 0" />
       <geometry>
             <cylinder radius="${shoulder_pan_width}" length="${shoulder_pan_len}"/>
@@ -160,5 +163,5 @@
     </visual>
     <collision>
-      <origin xyz="-0.002 0 -0.000" rpy="${M_PI/2} ${M_PI} ${M_PI/2}" />
+      <origin xyz="-0.002 0 0.04" rpy="0 ${M_PI/2} 0" />
       <geometry>
            <box size="${shoulder_pitch_len} ${shoulder_pitch_width} ${shoulder_pitch_height}" />
@@ -193,5 +196,5 @@
     </visual>
     <collision>
-      <origin xyz="-0.035 0.0 0.0" rpy="${M_PI} ${M_PI/2} ${M_PI/2}" />
+      <origin xyz="-0.035 0.0 -0.0" rpy="0 ${M_PI/2} 0" />
       <geometry>
             <cylinder radius="${elbow_roll_width}" length="${elbow_roll_len}"/>
@@ -226,5 +229,5 @@
     </visual>
     <collision>
-      <origin xyz="0.0 0 0" rpy="${M_PI/2} 0 ${M_PI/2+M_PI}" />
+      <origin xyz="0 0 -0.12" rpy="0 ${M_PI/2} 0" />
       <geometry>
        <box size="${elbow_pitch_len} ${elbow_pitch_width} ${elbow_pitch_height}" />
@@ -258,5 +261,5 @@
     </visual>
     <collision>
-      <origin xyz="0 0 0" rpy="0 ${M_PI/2} ${M_PI/2}" />
+      <origin xyz="0 0 0" rpy="0 ${M_PI/2} 0" />
       <geometry>
            <cylinder radius="${elbow_roll_width}" length="${elbow_roll_len}"/>
@@ -291,5 +294,5 @@
     </visual>
     <collision>
-      <origin xyz="0 0 0" rpy="${M_PI} -${M_PI/2} 0" />
+      <origin xyz="0 0 0.04 " rpy="0 ${M_PI/2} 0" />
       <geometry>
           <box size="${wrist_pitch_len} ${wrist_pitch_width} ${wrist_pitch_height}" />
@@ -324,5 +327,5 @@
     </visual>
     <collision>
-      <origin xyz="0 0 0" rpy="0 0 0" />
+      <origin xyz="0 0 0" rpy="0 ${M_PI/2} 0" />
       <geometry>
             <cylinder radius="${gripper_roll_width}" length="${gripper_roll_len}"/>

File: urdf/diff_wheeled_robot.xacro (robot description, xacro)
@@ -11,4 +11,7 @@
   <material name="White">
     <color rgba="1.0 1.0 1.0 1.0"/>
+  </material>
+  <material name="Blue">
+    <color rgba="0.0 0.0 0.8 1.0"/>
   </material>
   <!-- PROPERTY LIST -->
@@ -21,15 +24,15 @@
   <property name="base_height" value="0.02" />
   <property name="base_radius" value="0.15" />
-  <property name="base_mass" value="35" /> <!-- in kg-->
+  <property name="base_mass" value="5" /> <!-- in kg-->
   <!-- caster wheel radius and height -->
   <!-- caster wheel mass -->
   <property name="caster_f_height" value="0.04" />
-  <property name="caster_f_radius" value="0.008" />
-  <property name="caster_f_mass" value="35" /> <!-- in kg-->
+  <property name="caster_f_radius" value="0.025" />
+  <property name="caster_f_mass" value="0.5" /> <!-- in kg-->
   <!-- caster wheel radius and height -->
   <!-- caster wheel mass -->
   <property name="caster_b_height" value="0.04" />
-  <property name="caster_b_radius" value="0.008" />
-  <property name="caster_b_mass" value="35" /> <!-- in kg-->
+  <property name="caster_b_radius" value="0.025" />
+  <property name="caster_b_mass" value="0.5" /> <!-- in kg-->
   <!-- Wheels -->
 <!--  <property name="wheel_radius" value="0.2" />
@@ -39,4 +42,6 @@
   <property name="base_y_origin_to_wheel_origin" value="0.3" />
   <property name="base_z_origin_to_wheel_origin" value="0.0" />
+  <!-- Hokuyo Laser scanner -->
+  <property name="hokuyo_size" value="0.05" />
   <!-- Macro for calculating inertia of cylinder -->
   <macro name="cylinder_inertia" params="m r h">
@@ -99,4 +104,29 @@
   <wheel fb="front" lr="right" parent="base_link" translateX="0" translateY="-0.5" flipY="-1"/>
   <wheel fb="front" lr="left" parent="base_link" translateX="0" translateY="0.5" flipY="-1"/>
+<!--Caster front  -->
+    <link name="caster_front_link">
+    <visual>
+      <origin xyz="0 0.02 0" rpy="${M_PI/2} 0 0" />
+      <geometry>
+<!--       <mesh filename="package://mastering_ros_robot_description_pkg/meshes/caster_wheel.stl"/> -->
+<!--        <cylinder length="${caster_f_height}" radius="${caster_f_radius}" />  -->
+	<sphere radius="${caster_f_radius}" />
+      </geometry>
+      <material name="Black" />
+    </visual>
+      <collision>
+        <geometry>
+	<sphere radius="${caster_f_radius}" />
+        </geometry>
+      <origin xyz="0 0.02 0" rpy="${M_PI/2} 0 0" />
+      </collision>
+      <inertial>
+        <mass value="${caster_f_mass}" />
+        <origin xyz="0 0 0" />
+        <inertia ixx="0.001" ixy="0.0" ixz="0.0"
+                 iyy="0.001" iyz="0.0"
+                 izz="0.001" />
+      </inertial>
+    </link>
  <joint name="caster_front_joint" type="fixed">
       <parent link="base_link"/>
@@ -104,9 +134,15 @@
       <origin xyz="0.115 0.0 0.007" rpy="${-M_PI/2} 0 0"/>
     </joint>
-    <link name="caster_front_link">
-    <visual>
-      <origin xyz="0 0.02 0" rpy="${M_PI/2} 0 0" />
-      <geometry>
-          <cylinder length="${caster_f_height}" radius="${caster_f_radius}" />
+  <gazebo reference="caster_front_link">
+    <turnGravityOff>false</turnGravityOff>
+  </gazebo>
+<!--Caster back  -->
+    <link name="caster_back_link">
+    <visual>
+      <origin xyz="0.02 0.02 0 " rpy="${M_PI/2} 0 0" />
+      <geometry>
+<!--          <cylinder length="${caster_b_height}" radius="${caster_b_radius}" />   -->
+	<sphere radius="${caster_b_radius}" />
+<!--       <mesh filename="package://mastering_ros_robot_description_pkg/meshes/caster_wheel.stl"/>  -->
       </geometry>
       <material name="Black" />
@@ -114,10 +150,10 @@
       <collision>
         <geometry>
-          <cylinder length="${caster_f_height}" radius="${caster_f_radius}" />
+		<sphere radius="${caster_b_radius}" />
         </geometry>
-        <origin rpy="0 0 0" xyz="0 0 0"/>
+      <origin xyz="0 0.02 0 " rpy="${M_PI/2} 0 0" />
       </collision>
       <inertial>
-        <mass value="0.01" />
+        <mass value="${caster_b_mass}" />
         <origin xyz="0 0 0" />
         <inertia ixx="0.001" ixy="0.0" ixz="0.0"
@@ -131,25 +167,123 @@
       <origin xyz="-0.135 0.0 0.009" rpy="${-M_PI/2} 0 0"/>
     </joint>
-    <link name="caster_back_link">
-    <visual>
-      <origin xyz="0 0.02 0 " rpy="${M_PI/2} 0 0" />
-      <geometry>
-          <cylinder length="${caster_b_height}" radius="${caster_b_radius}" />
-      </geometry>
-      <material name="Black" />
-    </visual>
-      <collision>
-        <geometry>
-          <cylinder length="0.0176" radius="0.017"/>
-        </geometry>
-        <origin rpy="0 0 0" xyz="0 0 0"/>
-      </collision>
-      <inertial>
-        <mass value="0.01" />
-        <origin xyz="0 0 0" />
-        <inertia ixx="0.001" ixy="0.0" ixz="0.0"
-                 iyy="0.001" iyz="0.0"
-                 izz="0.001" />
-      </inertial>
-    </link>
+  <gazebo reference="caster_back_link">
+    <turnGravityOff>false</turnGravityOff>
+  </gazebo>
+  <!-- SENSORS -->
+  <!-- hokuyo -->
+  <link name="hokuyo_link">
+    <visual>
+      <origin xyz="0 0 0" rpy="0 0 0" />
+      <geometry>
+        <box size="${hokuyo_size} ${hokuyo_size} ${hokuyo_size}"/>
+      </geometry>
+      <material name="Blue" />
+    </visual>
+  </link>
+  <joint name="hokuyo_joint" type="fixed">
+    <origin xyz="${base_radius - hokuyo_size/2} 0 ${base_height+hokuyo_size/4}" rpy="0 0 0" />
+    <parent link="base_link"/>
+    <child link="hokuyo_link" />
+  </joint>
+  <gazebo reference="hokuyo_link">
+    <material>Gazebo/Blue</material>
+    <turnGravityOff>false</turnGravityOff>
+    <sensor type="ray" name="head_hokuyo_sensor">
+      <pose>${hokuyo_size/2} 0 0 0 0 0</pose>
+      <visualize>false</visualize>
+      <update_rate>40</update_rate>
+      <ray>
+        <scan>
+          <horizontal>
+            <samples>720</samples>
+            <resolution>1</resolution>
+            <min_angle>-1.570796</min_angle>
+            <max_angle>1.570796</max_angle>
+          </horizontal>
+        </scan>
+        <range>
+          <min>0.10</min>
+          <max>10.0</max>
+          <resolution>0.001</resolution>
+        </range>
+      </ray>
+      <plugin name="gazebo_ros_head_hokuyo_controller" filename="libgazebo_ros_laser.so">
+        <topicName>/scan</topicName>
+        <frameName>hokuyo_link</frameName>
+      </plugin>
+    </sensor>
+  </gazebo>
+  <!-- Kinect
+  <link name="kinect_link"/>
+  <joint name="kinect_joint" type="fixed">
+    <origin xyz="0.5 0 -0.1" rpy="0 0 0" />
+    <parent link="base_link"/>
+    <child link="kinect_link" />
+  </joint>
+  <sensor_kinect  parent="kinect_link"/> -->
+  <!-- DRIVE CONTROLLERS -->
+  <!-- Skid steer drive controller -->
+<!--
+  <gazebo>
+    <plugin name="gazebo_ros_control" filename="libgazebo_ros_control.so" />
+    <plugin name="skid_steer_drive_controller" filename="libgazebo_ros_skid_steer_drive.so">
+      <alwaysOn>1</alwaysOn>
+      <updateRate>100.0</updateRate>
+      <leftFrontJoint>front_left_wheel_joint</leftFrontJoint>
+      <rightFrontJoint>front_right_wheel_joint</rightFrontJoint>
+      <wheelSeparation>${base_height}</wheelSeparation>
+      <wheelDiameter>${2*wheel_radius}</wheelDiameter>
+      <torque>100</torque>
+      <broadcastTF>1</broadcastTF>
+      <odometryFrame>map</odometryFrame>
+      <commandTopic>cmd_vel</commandTopic>
+      <odometryTopic>odom</odometryTopic>
+      <robotBaseFrame>base_footprint</robotBaseFrame>
+    </plugin>
+  </gazebo>
+-->
+  <!-- Differential drive controller  -->
+  <gazebo>
+    <plugin name="differential_drive_controller_front" filename="libgazebo_ros_diff_drive.so">
+      <rosDebugLevel>Debug</rosDebugLevel>
+      <publishWheelTF>false</publishWheelTF>
+      <publishTf>1</publishTf>
+      <publishWheelJointState>true</publishWheelJointState>
+      <alwaysOn>true</alwaysOn>
+      <updateRate>100.0</updateRate>
+      <leftJoint>front_left_wheel_joint</leftJoint>
+      <rightJoint>front_right_wheel_joint</rightJoint>
+      <wheelSeparation>${2*base_radius}</wheelSeparation>
+      <wheelDiameter>${2*wheel_radius}</wheelDiameter>
+      <broadcastTF>1</broadcastTF>
+      <wheelTorque>100</wheelTorque>
+      <wheelAcceleration>1.8</wheelAcceleration>
+      <commandTopic>cmd_vel</commandTopic>
+      <odometryTopic>odom</odometryTopic>
+      <odometryFrame>map</odometryFrame>
+      <odometrySource>world</odometrySource>
+      <robotBaseFrame>base_footprint</robotBaseFrame>
+    </plugin>
+  </gazebo>
+<gazebo>
+    <plugin filename="libgazebo_ros_joint_state_publisher.so" name="joint_state_publisher">
+      <jointName>front_left_wheel_joint, front_right_wheel_joint</jointName>
+      <updateRate>10.0</updateRate>
+      <alwaysOn>true</alwaysOn>
+    </plugin>
+</gazebo>
+  <!-- GPS Sensor -->
+  <gazebo>
+    <plugin name="novatel_gps_sim" filename="libhector_gazebo_ros_gps.so">
+      <alwaysOn>1</alwaysOn>
+      <updateRate>10.0</updateRate>
+      <bodyName>base_footprint</bodyName>
+      <topicName>fix</topicName>
+      <velocityTopicName>fix_velocity</velocityTopicName>
+      <drift>5.0 5.0 5.0</drift>
+      <gaussianNoise>0.1 0.1 0.1</gaussianNoise>
+      <velocityDrift>0 0 0</velocityDrift>
+      <velocityGaussianNoise>0.1 0.1 0.1</velocityGaussianNoise>
+    </plugin>
+   </gazebo>
 </robot>
