Commit message: Update base.urdf

File: urdf/base.urdf (robot description, URDF)
Before this commit: robot demo_robot, 3 links, 2 joints
Links:
- link base_link: geometry collision box size=0.2 0.2 0.01; visual cylinder length=0.01 radius=0.1
- link first_link: geometry collision cylinder length=0.2 radius=0.04; visual cylinder length=0.2 radius=0.04
- link second_link: geometry collision box size=0.1 .1 .1; visual cylinder length=0.2 radius=0.04
Joints:
- joint joint_1: limit lower=-5 upper=6 effort=300 velocity=0.1 -> lower=-3.14 upper=3.14 effort=300 velocity=0.1; origin xyz=0 0 .1 -> xyz=0 0 0.1
- joint joint_2: axis 0 0 1 -> 0 1 0; limit lower=-5 upper=6 effort=300 velocity=0.1 -> lower=-4.64 upper=-1.5 effort=300 velocity=0.1; origin xyz=0 0 .1 -> xyz=0.01 -0.04 0.06

Commit message: Update base.urdf

File: urdf/base.urdf (robot description, URDF)
Before this commit: robot demo_robot, 3 links, 2 joints
Links:
- link base_link: geometry collision box size=0.2 0.2 0.01; visual cylinder length=0.01 radius=0.2
Joints:
- joint joint_2: origin xyz=0.01 -0.04 0.06 -> xyz=0 -0.04 0.06

Commit message: Update base.urdf

File: urdf/base.urdf (robot description, URDF)
Before this commit: robot demo_robot, 3 links, 2 joints
Links:
- link first_link: geometry collision cylinder length=0.2 radius=0.04; visual cylinder length=0.4 radius=0.04
- link second_link: geometry collision box size=0.1 .1 .1; visual cylinder length=0.4 radius=0.04
Joints:
- joint joint_2: origin xyz=0 -0.04 0.06 -> xyz=0 0 0.2
