Commit message: Update pan and tilt

File: urdf/pan_tilt.urdf (robot description, URDF)
Before this commit: robot demo_robot, 3 links, 2 joints
Links:
- link base_link: geometry collision cylinder length=0.03 radius=0.2; visual cylinder length=0.01 radius=0.2
- link first_link: geometry collision cylinder length=0.4 radius=0.06; visual cylinder length=0.4 radius=0.04
- link second_link: geometry collision cylinder length=0.4 radius=0.06; visual cylinder length=0.4 radius=0.04

Commit message: Update pan_tilt.urdf

File: urdf/pan_tilt.urdf (robot description, URDF)
Before this commit: robot demo_robot, 3 links, 2 joints
Links:
- removed link first_link
- removed link second_link
- added link pan_link; collision cylinder length=0.4 radius=0.06; visual cylinder length=0.4 radius=0.04
- added link tilt_link; collision cylinder length=0.4 radius=0.06; visual cylinder length=0.4 radius=0.04
Joints:
- removed joint joint_1
- removed joint joint_2
- added joint pan_joint: type revolute, parent base_link, child pan_link, origin xyz=0 0 0.1, axis 0 0 1, limit lower=-3.14 upper=3.14 effort=300 velocity=0.1
- added joint tilt_joint: type revolute, parent pan_link, child tilt_link, origin xyz=0 0 0.2, axis 0 1 0, limit lower=-4.64 upper=-1.5 effort=300 velocity=0.1

Commit message: Update inertial params

File: urdf/pan_tilt.urdf (robot description, URDF)
Before this commit: robot pan_tilt, 3 links, 2 joints
Links:
- link base_link: mass None -> 1
- link pan_link: mass None -> 1
- link tilt_link: mass None -> 1
