Commit message: Added gripper in urdf

File: urdf/seven_dof_arm.xacro (robot description, xacro)
@@ -408,8 +408,8 @@
     <type>transmission_interface/SimpleTransmission</type>
     <joint name="shoulder_pan_joint">
-      <hardwareInterface>EffortJointInterface</hardwareInterface>
-    </joint>
-    <actuator name="motor1">
-      <hardwareInterface>EffortJointInterface</hardwareInterface>
+      <hardwareInterface>hardware_interface/PositionJointInterface</hardwareInterface>
+    </joint>
+    <actuator name="motor1">
+      <hardwareInterface>hardware_interface/PositionJointInterface</hardwareInterface>
       <mechanicalReduction>1</mechanicalReduction>
     </actuator>
@@ -418,8 +418,8 @@
     <type>transmission_interface/SimpleTransmission</type>
     <joint name="shoulder_pitch_joint">
-      <hardwareInterface>EffortJointInterface</hardwareInterface>
-    </joint>
-    <actuator name="motor1">
-      <hardwareInterface>EffortJointInterface</hardwareInterface>
+      <hardwareInterface>hardware_interface/PositionJointInterface</hardwareInterface>
+    </joint>
+    <actuator name="motor1">
+      <hardwareInterface>hardware_interface/PositionJointInterface</hardwareInterface>
       <mechanicalReduction>1</mechanicalReduction>
     </actuator>
@@ -428,8 +428,8 @@
     <type>transmission_interface/SimpleTransmission</type>
     <joint name="elbow_roll_joint">
-      <hardwareInterface>EffortJointInterface</hardwareInterface>
-    </joint>
-    <actuator name="motor1">
-      <hardwareInterface>EffortJointInterface</hardwareInterface>
+      <hardwareInterface>hardware_interface/PositionJointInterface</hardwareInterface>
+    </joint>
+    <actuator name="motor1">
+      <hardwareInterface>hardware_interface/PositionJointInterface</hardwareInterface>
       <mechanicalReduction>1</mechanicalReduction>
     </actuator>
@@ -438,8 +438,8 @@
     <type>transmission_interface/SimpleTransmission</type>
     <joint name="elbow_pitch_joint">
-      <hardwareInterface>EffortJointInterface</hardwareInterface>
-    </joint>
-    <actuator name="motor1">
-      <hardwareInterface>EffortJointInterface</hardwareInterface>
+      <hardwareInterface>hardware_interface/PositionJointInterface</hardwareInterface>
+    </joint>
+    <actuator name="motor1">
+      <hardwareInterface>hardware_interface/PositionJointInterface</hardwareInterface>
       <mechanicalReduction>1</mechanicalReduction>
     </actuator>
@@ -448,8 +448,8 @@
     <type>transmission_interface/SimpleTransmission</type>
     <joint name="wrist_roll_joint">
-      <hardwareInterface>EffortJointInterface</hardwareInterface>
-    </joint>
-    <actuator name="motor1">
-      <hardwareInterface>EffortJointInterface</hardwareInterface>
+      <hardwareInterface>hardware_interface/PositionJointInterface</hardwareInterface>
+    </joint>
+    <actuator name="motor1">
+      <hardwareInterface>hardware_interface/PositionJointInterface</hardwareInterface>
       <mechanicalReduction>1</mechanicalReduction>
     </actuator>
@@ -458,14 +458,34 @@
     <type>transmission_interface/SimpleTransmission</type>
     <joint name="wrist_pitch_joint">
-      <hardwareInterface>EffortJointInterface</hardwareInterface>
-    </joint>
-    <actuator name="motor1">
-      <hardwareInterface>EffortJointInterface</hardwareInterface>
-      <mechanicalReduction>1</mechanicalReduction>
-    </actuator>
-  </transmission>
-  <transmission name="tran1">
-    <type>transmission_interface/SimpleTransmission</type>
-    <joint name="gripper_finger_joint">
+      <hardwareInterface>hardware_interface/PositionJointInterface</hardwareInterface>
+    </joint>
+    <actuator name="motor1">
+      <hardwareInterface>hardware_interface/PositionJointInterface</hardwareInterface>
+      <mechanicalReduction>1</mechanicalReduction>
+    </actuator>
+  </transmission>
+  <transmission name="tran1">
+    <type>transmission_interface/SimpleTransmission</type>
+    <joint name="gripper_roll_joint">
+      <hardwareInterface>hardware_interface/PositionJointInterface</hardwareInterface>
+    </joint>
+    <actuator name="motor1">
+      <hardwareInterface>hardware_interface/PositionJointInterface</hardwareInterface>
+      <mechanicalReduction>1</mechanicalReduction>
+    </actuator>
+  </transmission>
+  <transmission name="tran1">
+    <type>transmission_interface/SimpleTransmission</type>
+    <joint name="finger_joint1">
+      <hardwareInterface>hardware_interface/PositionJointInterface</hardwareInterface>
+    </joint>
+    <actuator name="motor1">
+      <hardwareInterface>hardware_interface/PositionJointInterface</hardwareInterface>
+      <mechanicalReduction>1</mechanicalReduction>
+    </actuator>
+  </transmission>
+  <transmission name="tran1">
+    <type>transmission_interface/SimpleTransmission</type>
+    <joint name="finger_joint2">
       <hardwareInterface>hardware_interface/PositionJointInterface</hardwareInterface>
     </joint>

Commit message: Update urdf of main models

File: urdf/seven_dof_arm.xacro (robot description, xacro)
@@ -352,5 +352,4 @@
   </joint>
 <!-- ///////////////////////////////////////////////////////////////////////////////////////////////////////////////////// -->
-<!-- ///////////////////////////////////////////////////////////////////////////////////////////////////////////////////// -->
   <!-- LEFT GRIPPER AFT LINK -->
   <link name="gripper_finger_link1">
@@ -365,5 +364,5 @@
            <box size="${left_gripper_len} ${left_gripper_width} ${left_gripper_height}" />
       </geometry>
-      <material name="Black" />
+      <material name="White" />
     </visual>
   </link>

Commit message: Update xacro arm

File: urdf/seven_dof_arm.xacro (robot description, xacro)
@@ -51,4 +51,22 @@
   <property name="grasp_frame_width" value="0.02" />
   <property name="grasp_frame_height" value="0.02" />
+   <xacro:macro name="inertial_matrix" params="mass">
+      <inertial>
+      	<mass value="${mass}" />
+        <inertia ixx="1.0" ixy="0.0" ixz="0.0" iyy="0.5" iyz="0.0" izz="1.0" />
+      </inertial>
+   </xacro:macro>
+   <xacro:macro name="transmission_block" params="joint_name">
+	  <transmission name="tran1">
+	    <type>transmission_interface/SimpleTransmission</type>
+	    <joint name="${joint_name}">
+	      <hardwareInterface>PositionJointInterface</hardwareInterface>
+	    </joint>
+	    <actuator name="motor1">
+	      <hardwareInterface>PositionJointInterface</hardwareInterface>
+	      <mechanicalReduction>1</mechanicalReduction>
+	    </actuator>
+	  </transmission>
+   </xacro:macro>
 <!-- BOTTOM FIXED LINK
 This link is the base of the arm in which arm is placed
@@ -61,10 +79,4 @@
   </joint>
   <link name="bottom_link">
-<!--    <inertial>
-      <origin xyz=" 0 0 -0.017"/>
-      <mass value="100.0" />
-      <inertia  ixx="1.0" ixy="0.0"  ixz="0.0"  iyy="100.0"  iyz="0.0"  izz="1.0" />
-    </inertial>
--->
     <visual>
       <origin xyz=" 0 0 -0.04"  rpy="0 0 0"/>
@@ -87,9 +99,4 @@
   <!-- BASE LINK -->
   <link name="base_link">
-    <inertial>
-        <origin xyz="0 0 0" />
-        <mass value="1.0" />
-        <inertia  ixx="1.0" ixy="0.0"  ixz="0.0"  iyy="100.0"  iyz="0.0"  izz="1.0" />
-        </inertial>
     <visual>
       <origin xyz="0 0 0" rpy="${M_PI/2} 0 0" /> <!-- rotate PI/2 -->
@@ -105,4 +112,5 @@
       </geometry>
       </collision>>
+	<xacro:inertial_matrix mass="1"/>
   </link>
   <gazebo reference="base_link">
@@ -120,9 +128,4 @@
   <!-- SHOULDER PAN LINK -->
   <link name="shoulder_pan_link" >
-    <inertial>
-      <origin xyz="0 0 0" />
-      <mass value="1.0" />
-      <inertia  ixx="1.0" ixy="0.0"  ixz="0.0"  iyy="100.0"  iyz="0.0"  izz="1.0" />
-    </inertial>
     <visual>
       <origin xyz="0 0 0" rpy="0 ${M_PI/2} 0" />
@@ -138,4 +141,5 @@
       </geometry>
     </collision>
+	<xacro:inertial_matrix mass="1"/>
   </link>
   <gazebo reference="shoulder_pan_link">
@@ -153,9 +157,4 @@
   <!-- SHOULDER PITCH LINK -->
   <link name="shoulder_pitch_link" >
-    <inertial>
-      <origin xyz="-0.002 0 -0.000"  />
-      <mass value="1.0" />
-      <inertia  ixx="1.0" ixy="0.0"  ixz="0.0"  iyy="100.0"  iyz="0.0"  izz="1.0" />
-    </inertial>
     <visual>
       <origin xyz="-0.002 0 0.04" rpy="0 ${M_PI/2} 0" />
@@ -171,4 +170,5 @@
       </geometry>
     </collision>
+	<xacro:inertial_matrix mass="1"/>
   </link>
   <gazebo reference="shoulder_pitch_link">
@@ -186,9 +186,4 @@
   <!-- ELBOW ROLL LINK -->
   <link name="elbow_roll_link" >
-    <inertial>
-      <origin xyz="-0.035 0.0 0.0"  />
-      <mass value="1.0" />
-      <inertia  ixx="1.0" ixy="0.0"  ixz="0.0"  iyy="100.0"  iyz="0.0"  izz="1.0" />
-    </inertial>
     <visual>
       <origin xyz="-0.015 0.0 -0.0" rpy="0 ${M_PI/2} 0" />
@@ -204,4 +199,5 @@
       </geometry>
     </collision>
+	<xacro:inertial_matrix mass="1"/>
   </link>
   <gazebo reference="elbow_roll_link">
@@ -219,9 +215,4 @@
   <!-- ELBOW PITCH LINK -->
   <link name="elbow_pitch_link" >
-    <inertial>
-      <origin xyz="0.0 0 0"  />
-      <mass value="1.0" />
-      <inertia  ixx="1.0" ixy="0.0"  ixz="0.0"  iyy="100.0"  iyz="0.0"  izz="1.0" />
-    </inertial>
     <visual>
       <origin xyz="0 0 -0.12" rpy="0 ${M_PI/2} 0" />
@@ -237,4 +228,5 @@
       </geometry>
     </collision>
+	<xacro:inertial_matrix mass="1"/>
   </link>
   <gazebo reference="elbow_pitch_link">
@@ -251,9 +243,4 @@
   <!-- WRIST ROLL LINK -->
   <link name="wrist_roll_link" >
-    <inertial>
-      <origin xyz="0 0 0"  />
-      <mass value="1.0" />
-      <inertia  ixx="1.0" ixy="0.0"  ixz="0.0"  iyy="100.0"  iyz="0.0"  izz="1.0" />
-    </inertial>
     <visual>
       <origin xyz="0 0 0" rpy="0 ${M_PI/2} 0" />
@@ -269,4 +256,5 @@
       </geometry>
     </collision>
+	<xacro:inertial_matrix mass="1"/>
   </link>
   <gazebo reference="wrist_roll_link">
@@ -284,9 +272,4 @@
   <!-- WRIST PITCH LINK -->
   <link name="wrist_pitch_link">
-    <inertial>
-      <origin xyz="0 0 0"  />
-      <mass value="1.0" />
-      <inertia  ixx="1.0" ixy="0.0"  ixz="0.0"  iyy="100.0"  iyz="0.0"  izz="1.0" />
-    </inertial>
     <visual>
       <origin xyz="0 0 0.04" rpy="0 ${M_PI/2} 0" />
@@ -302,4 +285,5 @@
       </geometry>
     </collision>
+	<xacro:inertial_matrix mass="1"/>
   </link>
   <gazebo reference="wrist_pitch_link">
@@ -317,9 +301,4 @@
   <!-- GRIPPER ROLL LINK -->
   <link name="gripper_roll_link">
-    <inertial>
-      <origin xyz="0 0 0" />
-      <mass value="1.0" />
-      <inertia  ixx="1.0" ixy="0.0"  ixz="0.0"  iyy="100.0"  iyz="0.0"  izz="1.0" />
-    </inertial>
     <visual>
       <origin xyz="0 0 0" rpy="0 ${M_PI/2} 0" />
@@ -335,4 +314,5 @@
       </geometry>
     </collision>
+	<xacro:inertial_matrix mass="1"/>
   </link>
   <gazebo reference="gripper_roll_link">
@@ -354,10 +334,5 @@
   <!-- LEFT GRIPPER AFT LINK -->
   <link name="gripper_finger_link1">
-    <inertial>
-      <origin xyz="0 0 0"  />
-      <mass value="0.01" />
-      <inertia  ixx="1.0" ixy="0.0"  ixz="0.0"  iyy="100.0"  iyz="0.0"  izz="1.0" />
-    </inertial>
-    <visual>
+     <visual>
       <origin xyz="0.04 -0.03 0"/>
       <geometry>
@@ -366,4 +341,5 @@
       <material name="White" />
     </visual>
+	<xacro:inertial_matrix mass="1"/>
   </link>
   <gazebo reference="l_gripper_aft_link">
@@ -383,9 +359,4 @@
   <!-- RIGHT GRIPPER AFT LINK -->
   <link name="gripper_finger_link2">
-    <inertial>
-      <origin xyz="0.0 0.0 0"  />
-      <mass value="1.0" />
-      <inertia  ixx="1.0" ixy="0.0"  ixz="0.0"  iyy="100.0"  iyz="0.0"  izz="1.0" />
-    </inertial>
     <visual>
       <origin xyz="0.04 0.03 0"/>
@@ -395,4 +366,5 @@
       <material name="White" />
     </visual>
+	<xacro:inertial_matrix mass="1"/>
   </link>
   <gazebo reference="r_gripper_aft_link">
@@ -423,94 +395,13 @@
 <!-- ///////////////////////////////////////////////////////////////////////////////////////////////////////////////////// -->
   <!-- Transmissions for ROS Control -->
-  <transmission name="tran1">
-    <type>transmission_interface/SimpleTransmission</type>
-    <joint name="shoulder_pan_joint">
-      <hardwareInterface>PositionJointInterface</hardwareInterface>
-    </joint>
-    <actuator name="motor1">
-      <hardwareInterface>PositionJointInterface</hardwareInterface>
-      <mechanicalReduction>1</mechanicalReduction>
-    </actuator>
-  </transmission>
-  <transmission name="tran1">
-    <type>transmission_interface/SimpleTransmission</type>
-    <joint name="shoulder_pitch_joint">
-      <hardwareInterface>PositionJointInterface</hardwareInterface>
-    </joint>
-    <actuator name="motor1">
-      <hardwareInterface>PositionJointInterface</hardwareInterface>
-      <mechanicalReduction>1</mechanicalReduction>
-    </actuator>
-  </transmission>
-  <transmission name="tran1">
-    <type>transmission_interface/SimpleTransmission</type>
-    <joint name="elbow_roll_joint">
-      <hardwareInterface>PositionJointInterface</hardwareInterface>
-    </joint>
-    <actuator name="motor1">
-      <hardwareInterface>PositionJointInterface</hardwareInterface>
-      <mechanicalReduction>1</mechanicalReduction>
-    </actuator>
-  </transmission>
-  <transmission name="tran1">
-    <type>transmission_interface/SimpleTransmission</type>
-    <joint name="elbow_pitch_joint">
-      <hardwareInterface>PositionJointInterface</hardwareInterface>
-    </joint>
-    <actuator name="motor1">
-      <hardwareInterface>PositionJointInterface</hardwareInterface>
-      <mechanicalReduction>1</mechanicalReduction>
-    </actuator>
-  </transmission>
-  <transmission name="tran1">
-    <type>transmission_interface/SimpleTransmission</type>
-    <joint name="wrist_roll_joint">
-      <hardwareInterface>PositionJointInterface</hardwareInterface>
-    </joint>
-    <actuator name="motor1">
-      <hardwareInterface>PositionJointInterface</hardwareInterface>
-      <mechanicalReduction>1</mechanicalReduction>
-    </actuator>
-  </transmission>
-  <transmission name="tran1">
-    <type>transmission_interface/SimpleTransmission</type>
-    <joint name="wrist_pitch_joint">
-      <hardwareInterface>PositionJointInterface</hardwareInterface>
-    </joint>
-    <actuator name="motor1">
-      <hardwareInterface>PositionJointInterface</hardwareInterface>
-      <mechanicalReduction>1</mechanicalReduction>
-    </actuator>
-  </transmission>
-  <transmission name="tran1">
-    <type>transmission_interface/SimpleTransmission</type>
-    <joint name="gripper_roll_joint">
-      <hardwareInterface>PositionJointInterface</hardwareInterface>
-    </joint>
-    <actuator name="motor1">
-      <hardwareInterface>PositionJointInterface</hardwareInterface>
-      <mechanicalReduction>1</mechanicalReduction>
-    </actuator>
-  </transmission>
-  <transmission name="tran1">
-    <type>transmission_interface/SimpleTransmission</type>
-    <joint name="finger_joint1">
-      <hardwareInterface>PositionJointInterface</hardwareInterface>
-    </joint>
-    <actuator name="motor1">
-      <hardwareInterface>PositionJointInterface</hardwareInterface>
-      <mechanicalReduction>1</mechanicalReduction>
-    </actuator>
-  </transmission>
-  <transmission name="tran1">
-    <type>transmission_interface/SimpleTransmission</type>
-    <joint name="finger_joint2">
-      <hardwareInterface>PositionJointInterface</hardwareInterface>
-    </joint>
-    <actuator name="motor1">
-      <hardwareInterface>PositionJointInterface</hardwareInterface>
-      <mechanicalReduction>1</mechanicalReduction>
-    </actuator>
-  </transmission>
+   <xacro:transmission_block joint_name="shoulder_pan_joint"/>
+   <xacro:transmission_block joint_name="shoulder_pitch_joint"/>
+   <xacro:transmission_block joint_name="elbow_roll_joint"/>
+   <xacro:transmission_block joint_name="elbow_pitch_joint"/>
+   <xacro:transmission_block joint_name="wrist_roll_joint"/>
+   <xacro:transmission_block joint_name="wrist_pitch_joint"/>
+   <xacro:transmission_block joint_name="gripper_roll_joint"/>
+   <xacro:transmission_block joint_name="finger_joint1"/>
+   <xacro:transmission_block joint_name="finger_joint2"/>
   <!-- Define arm with gripper mounted on a base -->
   <xacro:base name="base"/>
