Commit message: Updated urdf model

File: urdf/bkup/7_dof_arm.xacro (robot description, xacro)
@@ -36,18 +36,14 @@
   <property name="wrist_pitch_height" value="0.04" />
   <!-- Gripper roll link properties -->
-  <property name="gripper_roll_width" value="0.04" />
-  <property name="gripper_roll_len" value="0.02" />
+  <property name="gripper_roll_width" value="0.02" />
+  <property name="gripper_roll_len" value="0.04" />
   <!-- Left gripper -->
-  <property name="left_gripper_len" value="0.08" />
-  <property name="left_gripper_width" value="0.01" />
+  <property name="left_gripper_len" value="0.02" />
+  <property name="left_gripper_width" value="0.08" />
   <property name="left_gripper_height" value="0.01" />
   <!-- Right gripper -->
-  <property name="right_gripper_len" value="0.08" />
-  <property name="right_gripper_width" value="0.01" />
+  <property name="right_gripper_len" value="0.02" />
+  <property name="right_gripper_width" value="0.08" />
   <property name="right_gripper_height" value="0.01" />
-  <!-- Right gripper -->
-  <property name="grasp_frame_len" value="0.02" />
-  <property name="grasp_frame_width" value="0.02" />
-  <property name="grasp_frame_height" value="0.02" />
 <!-- BOTTOM FIXED LINK
 This link is the base of the arm in which arm is placed
@@ -79,18 +75,15 @@
       </collision>>
   </link>
-<!--
   <gazebo reference="bottom_link">
     <material>Gazebo/White</material>
   </gazebo>
--->
 <!-- ///////////////////////////////////////////////////////////////////////////////////////////////////////////////////// -->
   <!-- BASE LINK -->
   <link name="base_link">
-<!--    <inertial>
+    <inertial>
         <origin xyz="0 0 0" />
         <mass value="1.0" />
         <inertia  ixx="1.0" ixy="0.0"  ixz="0.0"  iyy="100.0"  iyz="0.0"  izz="1.0" />
         </inertial>
--->
     <visual>
       <origin xyz="0 0 0" rpy="${M_PI/2} 0 0" /> <!-- rotate PI/2 -->
@@ -340,27 +333,26 @@
     <material>Gazebo/Red</material>
   </gazebo>
-<!-- Joint between wrist roll and finger 1 -->
-  <joint name="finger_joint1" type="prismatic">
+  <joint name="gripper_finger_joint" type="revolute">
     <parent link="gripper_roll_link"/>
-    <child link="gripper_finger_link1"/>
-    <origin xyz="0.0 0 0" />
-    <axis xyz="0 1 0" />
-      <limit effort="1" lower="0" upper="0.03" velocity="1.0"/>
+    <child link="gripper_finger_link"/>
+    <origin xyz="0.026 .017 0" rpy="${1.04*M_PI} ${M_PI/2} ${34.58*M_PI/180}" />
+    <axis xyz="1 0 0" />
+    <limit effort="300" velocity="1" lower="${53*M_PI/180}" upper="${0*M_PI/180}"/>
     <dynamics damping="50" friction="1"/>
   </joint>
 <!-- ///////////////////////////////////////////////////////////////////////////////////////////////////////////////////// -->
   <!-- LEFT GRIPPER AFT LINK -->
-  <link name="gripper_finger_link1">
+  <link name="gripper_finger_link">
     <inertial>
       <origin xyz="0 0 0"  />
-      <mass value="0.01" />
-      <inertia  ixx="1.0" ixy="0.0"  ixz="0.0"  iyy="100.0"  iyz="0.0"  izz="1.0" />
-    </inertial>
-    <visual>
-      <origin xyz="0.04 -0.03 0"/>
+      <mass value="1.0" />
+      <inertia  ixx="1.0" ixy="0.0"  ixz="0.0"  iyy="100.0"  iyz="0.0"  izz="1.0" />
+    </inertial>
+    <visual>
+      <origin xyz="0 0 0" rpy="${M_PI/2} 0 0 " />
       <geometry>
            <box size="${left_gripper_len} ${left_gripper_width} ${left_gripper_height}" />
       </geometry>
-      <material name="Black" />
+      <material name="White" />
     </visual>
   </link>
@@ -368,24 +360,23 @@
     <material>Gazebo/White</material>
   </gazebo>
-<!-- Joint between Wrist roll and finger 2 -->
-  <joint name="finger_joint2" type="prismatic">
+  <joint name="r_gripper_aft_joint" type="revolute">
     <parent link="gripper_roll_link"/>
-    <child link="gripper_finger_link2"/>
-    <origin xyz="0.0 0 0" />
-    <axis xyz="0 1 0" />
-    <limit effort="1" lower="-0.03" upper="0" velocity="1.0"/>
-<!--    <mimic joint="gripper_finger_joint" multiplier="-1.0" offset="0.0" /> -->
+    <child link="r_gripper_aft_link"/>
+    <origin xyz="0.026 -0.011  0" rpy="${1.345*M_PI} ${M_PI/2} ${34.58*M_PI/180}" />
+    <axis xyz="1 0 0" />
+    <limit effort="300" velocity="1" lower="-3.14" upper="3.14" />
+    <mimic joint="gripper_finger_joint" multiplier="-1.0" offset="0.0" />
     <dynamics damping="50" friction="1"/>
   </joint>
 <!-- ///////////////////////////////////////////////////////////////////////////////////////////////////////////////////// -->
   <!-- RIGHT GRIPPER AFT LINK -->
-  <link name="gripper_finger_link2">
-    <inertial>
-      <origin xyz="0.0 0.0 0"  />
-      <mass value="1.0" />
-      <inertia  ixx="1.0" ixy="0.0"  ixz="0.0"  iyy="100.0"  iyz="0.0"  izz="1.0" />
-    </inertial>
-    <visual>
-      <origin xyz="0.04 0.03 0"/>
+  <link name="r_gripper_aft_link">
+    <inertial>
+      <origin xyz="0 0 0"  />
+      <mass value="1.0" />
+      <inertia  ixx="1.0" ixy="0.0"  ixz="0.0"  iyy="100.0"  iyz="0.0"  izz="1.0" />
+    </inertial>
+    <visual>
+      <origin xyz="0 0 0" rpy="${M_PI/2} 0 0 " />
       <geometry>
           <box size="${right_gripper_len} ${right_gripper_width} ${right_gripper_height}" />
@@ -397,25 +388,4 @@
     <material>Gazebo/White</material>
   </gazebo>
-    <!-- Grasping frame -->
-    <link name="grasping_frame">
-      <inertial>
-        <origin xyz="0 0 0" rpy="0 0 0"/>
-        <mass value="0.0001"/>
-        <cuboid_inertia mass="0.0001" x="0.001" y="0.001" z="0.001"/>
-        <inertia  ixx="1.0" ixy="0.0"  ixz="0.0"  iyy="100.0"  iyz="0.0"  izz="1.0" />
-      </inertial>
-    <visual>
-      <origin xyz="0 0 0"/>
-      <geometry>
-          <box size="${grasp_frame_len} ${grasp_frame_width} ${grasp_frame_height}" />
-      </geometry>
-      <material name="White" />
-    </visual>
-    </link>
-    <joint name="grasping_frame_joint" type="fixed">
-      <parent link="gripper_roll_link"/>
-      <child link="grasping_frame"/>
-      <origin xyz="0.08 0 0" rpy="0 0 0"/>
-    </joint>
 <!-- ///////////////////////////////////////////////////////////////////////////////////////////////////////////////////// -->
   <!-- Transmissions for ROS Control -->
@@ -423,8 +393,8 @@
     <type>transmission_interface/SimpleTransmission</type>
     <joint name="shoulder_pan_joint">
-      <hardwareInterface>PositionJointInterface</hardwareInterface>
-    </joint>
-    <actuator name="motor1">
-      <hardwareInterface>PositionJointInterface</hardwareInterface>
+      <hardwareInterface>EffortJointInterface</hardwareInterface>
+    </joint>
+    <actuator name="motor1">
+      <hardwareInterface>EffortJointInterface</hardwareInterface>
       <mechanicalReduction>1</mechanicalReduction>
     </actuator>
@@ -433,8 +403,8 @@
     <type>transmission_interface/SimpleTransmission</type>
     <joint name="shoulder_pitch_joint">
-      <hardwareInterface>PositionJointInterface</hardwareInterface>
-    </joint>
-    <actuator name="motor1">
-      <hardwareInterface>PositionJointInterface</hardwareInterface>
+      <hardwareInterface>EffortJointInterface</hardwareInterface>
+    </joint>
+    <actuator name="motor1">
+      <hardwareInterface>EffortJointInterface</hardwareInterface>
       <mechanicalReduction>1</mechanicalReduction>
     </actuator>
@@ -443,8 +413,8 @@
     <type>transmission_interface/SimpleTransmission</type>
     <joint name="elbow_roll_joint">
-      <hardwareInterface>PositionJointInterface</hardwareInterface>
-    </joint>
-    <actuator name="motor1">
-      <hardwareInterface>PositionJointInterface</hardwareInterface>
+      <hardwareInterface>EffortJointInterface</hardwareInterface>
+    </joint>
+    <actuator name="motor1">
+      <hardwareInterface>EffortJointInterface</hardwareInterface>
       <mechanicalReduction>1</mechanicalReduction>
     </actuator>
@@ -453,8 +423,8 @@
     <type>transmission_interface/SimpleTransmission</type>
     <joint name="elbow_pitch_joint">
-      <hardwareInterface>PositionJointInterface</hardwareInterface>
-    </joint>
-    <actuator name="motor1">
-      <hardwareInterface>PositionJointInterface</hardwareInterface>
+      <hardwareInterface>EffortJointInterface</hardwareInterface>
+    </joint>
+    <actuator name="motor1">
+      <hardwareInterface>EffortJointInterface</hardwareInterface>
       <mechanicalReduction>1</mechanicalReduction>
     </actuator>
@@ -463,8 +433,8 @@
     <type>transmission_interface/SimpleTransmission</type>
     <joint name="wrist_roll_joint">
-      <hardwareInterface>PositionJointInterface</hardwareInterface>
-    </joint>
-    <actuator name="motor1">
-      <hardwareInterface>PositionJointInterface</hardwareInterface>
+      <hardwareInterface>EffortJointInterface</hardwareInterface>
+    </joint>
+    <actuator name="motor1">
+      <hardwareInterface>EffortJointInterface</hardwareInterface>
       <mechanicalReduction>1</mechanicalReduction>
     </actuator>
@@ -473,8 +443,8 @@
     <type>transmission_interface/SimpleTransmission</type>
     <joint name="wrist_pitch_joint">
-      <hardwareInterface>PositionJointInterface</hardwareInterface>
-    </joint>
-    <actuator name="motor1">
-      <hardwareInterface>PositionJointInterface</hardwareInterface>
+      <hardwareInterface>EffortJointInterface</hardwareInterface>
+    </joint>
+    <actuator name="motor1">
+      <hardwareInterface>EffortJointInterface</hardwareInterface>
       <mechanicalReduction>1</mechanicalReduction>
     </actuator>
@@ -483,28 +453,18 @@
     <type>transmission_interface/SimpleTransmission</type>
     <joint name="gripper_roll_joint">
-      <hardwareInterface>PositionJointInterface</hardwareInterface>
-    </joint>
-    <actuator name="motor1">
-      <hardwareInterface>PositionJointInterface</hardwareInterface>
-      <mechanicalReduction>1</mechanicalReduction>
-    </actuator>
-  </transmission>
-  <transmission name="tran1">
-    <type>transmission_interface/SimpleTransmission</type>
-    <joint name="finger_joint1">
-      <hardwareInterface>PositionJointInterface</hardwareInterface>
-    </joint>
-    <actuator name="motor1">
-      <hardwareInterface>PositionJointInterface</hardwareInterface>
-      <mechanicalReduction>1</mechanicalReduction>
-    </actuator>
-  </transmission>
-  <transmission name="tran1">
-    <type>transmission_interface/SimpleTransmission</type>
-    <joint name="finger_joint2">
-      <hardwareInterface>PositionJointInterface</hardwareInterface>
-    </joint>
-    <actuator name="motor1">
-      <hardwareInterface>PositionJointInterface</hardwareInterface>
+      <hardwareInterface>EffortJointInterface</hardwareInterface>
+    </joint>
+    <actuator name="motor1">
+      <hardwareInterface>EffortJointInterface</hardwareInterface>
+      <mechanicalReduction>1</mechanicalReduction>
+    </actuator>
+  </transmission>
+  <transmission name="tran1">
+    <type>transmission_interface/SimpleTransmission</type>
+    <joint name="gripper_finger_joint">
+      <hardwareInterface>EffortJointInterface</hardwareInterface>
+    </joint>
+    <actuator name="motor1">
+      <hardwareInterface>EffortJointInterface</hardwareInterface>
       <mechanicalReduction>1</mechanicalReduction>
     </actuator>
@@ -513,7 +473,5 @@
   <gazebo>
     <plugin name="gazebo_ros_control" filename="libgazebo_ros_control.so">
-      <robotNamespace>/seven_arm</robotNamespace>
-      <robotSimType>gazebo_ros_control/DefaultRobotHWSim</robotSimType>
-      <controlPeriod>0.001</controlPeriod>
+      <robotNamespace>/seven_dof_arm</robotNamespace>
     </plugin>
   </gazebo>
